File: Kicad/PMOD SPI Memory.kicad_pcb (KiCad board)
At the start: 2 copper layers, 49.5 x 20.3 mm, 6 parts, among them J1 Pmod peripheral SPI, U1 SPI Memory

Commit message: Small tweaks.
Other:
- board text added: "${COMMENT1}"
- board text added: "${COMPANY}"
- board text added: "${ISSUE_DATE}, ${REVISION}"
- board text removed: "2023-03-31, V1.0"
- board text removed: "https://github.com/atoomnetmarc/PMOD-SPI-Memory"
Changed lines of the file:
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@@
   (title_block
     (title "PMOD SPI Memory")
-    (date "2023-03-31")
+    (date "2023-04-01")
     (rev "V1.0")
     (company "https://github.com/atoomnetmarc/PMOD-SPI-Memory")
+    (comment 1 "Apache License, version 2.0")
   )
   (layers
@@
     )
   )
-  (gr_rect (start 114.962856 116.84) (end 135.282856 113.03)
+  (gr_rect (start 125.73 113.03) (end 146.05 116.84)
     (stroke (width 0.15) (type solid)) (fill solid) (layer "B.SilkS"))
   (gr_rect (start 131.445 113.03) (end 145.415 116.84)
@@
   (gr_line (start 97.79 118.11) (end 147.32 118.11)
     (stroke (width 0.1) (type default)) (layer "Edge.Cuts"))
-  (gr_text "Partnumber:" (at 135.89 115.57) (layer "B.SilkS")
+  (gr_text "${COMMENT1}" (at 99.06 116.84) (layer "B.SilkS")
     (effects (font (size 1 1) (thickness 0.15)) (justify right mirror))
   )
+  (gr_text "Partnumber:" (at 146.05 111.76) (layer "B.SilkS")
+    (effects (font (size 1 1) (thickness 0.15)) (justify left mirror))
+  )
   (gr_text "{dblquote}Ah, memory, the faulty tape recorder of the mind.{dblquote}" (at 122.555 99.695) (layer "B.SilkS")
     (effects (font (face "Segoe Script") (size 1.2 1.2) (thickness 0.15)) (justify mirror))
@@
     (effects (font (size 1 1) (thickness 0.15)) (justify right))
   )
-  (gr_text "MISO" (at 106.045 106.68) (layer "F.SilkS")
-    (effects (font (size 1 1) (thickness 0.15)))
+  (gr_text "MISO" (at 104.14 106.68) (layer "F.SilkS")
+    (effects (font (size 1 1) (thickness 0.15)) (justify left))
   )
-  (gr_text "2023-03-31, V1.0" (at 114.3 116.84) (layer "F.SilkS")
+  (gr_text "${ISSUE_DATE}, ${REVISION}" (at 114.3 116.84) (layer "F.SilkS")
     (effects (font (size 1 1) (thickness 0.15)))
   )
-  (gr_text "~{CS}" (at 106.045 101.6) (layer "F.SilkS")
-    (effects (font (size 1 1) (thickness 0.15)))
+  (gr_text "~{CS}" (at 104.14 101.6) (layer "F.SilkS")
+    (effects (font (size 1 1) (thickness 0.15)) (justify left))
   )
   (gr_text "Capacity:" (at 130.81 115.57) (layer "F.SilkS")
     (effects (font (size 1 1) (thickness 0.15)) (justify right))
   )
-  (gr_text "https://github.com/atoomnetmarc/PMOD-SPI-Memory" (at 121.92 99.06) (layer "F.SilkS")
+  (gr_text "${COMPANY}" (at 121.92 99.06) (layer "F.SilkS")
     (effects (font (size 1 1) (thickness 0.15)))
   )
-  (gr_text "VCC" (at 106.045 114.3) (layer "F.SilkS")
-    (effects (font (size 1 1) (thickness 0.15)))
+  (gr_text "VCC" (at 104.14 114.3) (layer "F.SilkS")
+    (effects (font (size 1 1) (thickness 0.15)) (justify left))
   )
-  (gr_text "SCK" (at 106.045 109.22) (layer "F.SilkS")
-    (effects (font (size 1 1) (thickness 0.15)))
+  (gr_text "SCK" (at 104.14 109.22) (layer "F.SilkS")
+    (effects (font (size 1 1) (thickness 0.15)) (justify left))
   )
-  (gr_text "GND" (at 106.045 111.76) (layer "F.SilkS")
-    (effects (font (size 1 1) (thickness 0.15)))
+  (gr_text "GND" (at 104.14 111.76) (layer "F.SilkS")
+    (effects (font (size 1 1) (thickness 0.15)) (justify left))
   )
-  (gr_text "MOSI" (at 106.045 104.14) (layer "F.SilkS")
-    (effects (font (size 1 1) (thickness 0.15)))
+  (gr_text "MOSI" (at 104.14 104.14) (layer "F.SilkS")
+    (effects (font (size 1 1) (thickness 0.15)) (justify left))
   )
   (gr_text "DRAM" (at 142.875 103.505) (layer "F.SilkS")
